File: Microarchitecture/Microarchitecture/RSA.kicad_sch (KiCad schematic)
At the start: 0 parts

Commit message: Updated timing diagrams, etc, control fsm and verified workings
Other:
- added sheet AXI_RECEIVE_MODULE (AXI_RECEIVE.kicad_sch)
- added sheet AXI_TRANSMIT_MODULE (AXI_TRANSMIT.kicad_sch)
- sheet RSA_STAGE_MODULE ports: added DCI, DCO, DPI, DPO, ILI, ILO, IPI, IPO, N; removed II, IL, IO, IP
- note added: "rsa_core"
Changed lines of the file:
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@@
 	(generator_version "8.0")
 	(paper "A4")
+	(rectangle
+		(start 76.2 50.8)
+		(end 215.9 114.3)
+		(stroke
+			(width 0.254)
+			(type default)
+		)
+		(fill
+			(type none)
+		)
+	)
+	(text "rsa_core"
+		(exclude_from_sim no)
+		(at 147.32 56.896 0)
+		(effects
+			(font
+				(size 2.54 2.54)
+				(thickness 0.508)
+				(bold yes)
+			)
+		)
+	)
 	(sheet
-		(at 60.96 73.66)
-		(size 33.02 17.78)
+		(at 177.8 63.5)
+		(size 25.4 44.45)
 		(fields_autoplaced yes)
 		(stroke
@@
 			(color 0 0 0 0.0000)
 		)
+		(property "Sheetname" "AXI_TRANSMIT_MODULE"
+			(at 177.8 62.7884 0)
+			(effects
+				(font
+					(size 1.27 1.27)
+				)
+				(justify left bottom)
+			)
+		)
+		(property "Sheetfile" "AXI_TRANSMIT.kicad_sch"
+			(at 177.8 108.5346 0)
+			(effects
+				(font
+					(size 1.27 1.27)
+				)
+				(justify left top)
+			)
+		)
+		(instances
+			(project "Microarchitecture"
+				(path "/7e18b03f-0dd8-4430-9873-65919f4f0c9c/21c2d8ae-34c8-4eeb-a025-0344b2d7e18d"
+					(page "7")
+				)
+			)
+		)
+	)
+	(sheet
+		(at 88.9 63.5)
+		(size 25.4 44.45)
+		(fields_autoplaced yes)
+		(stroke
+			(width 0.1524)
+			(type solid)
+		)
+		(fill
+			(color 0 0 0 0.0000)
+		)
+		(property "Sheetname" "AXI_RECEIVE_MODULE"
+			(at 88.9 62.7884 0)
+			(effects
+				(font
+					(size 1.27 1.27)
+				)
+				(justify left bottom)
+			)
+		)
+		(property "Sheetfile" "AXI_RECEIVE.kicad_sch"
+			(at 88.9 108.5346 0)
+			(effects
+				(font
+					(size 1.27 1.27)
+				)
+				(justify left top)
+			)
+		)
+		(instances
+			(project "Microarchitecture"
+				(path "/7e18b03f-0dd8-4430-9873-65919f4f0c9c/21c2d8ae-34c8-4eeb-a025-0344b2d7e18d"
+					(page "8")
+				)
+			)
+		)
+	)
+	(sheet
+		(at 129.54 76.2)
+		(size 33.02 17.78)
+		(stroke
+			(width 0.1524)
+			(type solid)
+		)
+		(fill
+			(color 0 0 0 0.0000)
+		)
 		(property "Sheetname" "RSA_STAGE_MODULE"
-			(at 60.96 72.9484 0)
+			(at 136.652 86.36 0)
 			(effects
 				(font
@@
 		)
 		(property "Sheetfile" "STAGE.kicad_sch"
-			(at 60.96 92.0246 0)
+			(at 129.54 94.5646 0)
 			(effects
 				(font
@@
 		)
 		(pin "ES" input
-			(at 82.55 73.66 90)
-			(effects
-				(font
-					(size 1.27 1.27)
-				)
-				(justify right)
-			)
-		)
-		(pin "IL" input
-			(at 93.98 87.63 0)
-			(effects
-				(font
-					(size 1.27 1.27)
-				)
-				(justify right)
-			)
-		)
-		(pin "IP" output
-			(at 60.96 87.63 180)
-			(effects
-				(font
-					(size 1.27 1.27)
-				)
-				(justify left)
-			)
-		)
-		(pin "IO" output
-			(at 93.98 81.28 0)
-			(effects
-				(font
-					(size 1.27 1.27)
-				)
-				(justify right)
-			)
-		)
-		(pin "II" input
-			(at 60.96 81.28 180)
-			(effects
-				(font
-					(size 1.27 1.27)
-				)
-				(justify left)
-			)
-		)
+			(at 149.86 76.2 90)
+			(effects
+				(font
+					(size 1.27 1.27)
+				)
+				(justify right)
+			)
+		)
+		(pin "IPO" output
+			(at 129.54 91.44 180)
+			(effects
+				(font
+					(size 1.27 1.27)
+				)
+				(justify left)
+			)
+		)
+		(pin "DCI" input
+			(at 129.54 83.82 180)
+			(effects
+				(font
+					(size 1.27 1.27)
+				)
+				(justify left)
+			)
+		)
+		(pin "ILI" input
+			(at 129.54 88.9 180)
+			(effects
+				(font
+					(size 1.27 1.27)
+				)
+				(justify left)
+			)
+		)
+		(pin "DPI" input
+			(at 129.54 81.28 180)
+			(effects
+				(font
+					(size 1.27 1.27)
+				)
+				(justify left)
+			)
+		)
+		(pin "N" input
+			(at 142.24 76.2 90)
+			(effects
+				(font
+					(size 1.27 1.27)
+				)
+				(justify right)
+			)
+		)
+		(pin "ILO" output
+			(at 162.56 88.9 0)
+			(effects
+				(font
+					(size 1.27 1.27)
+				)
+				(justify right)
+			)
+		)
+		(pin "DCO" output
+			(at 162.56 83.82 0)
+			(effects
+				(font
+					(size 1.27 1.27)
+				)
+				(justify right)
+			)
+		)
+		(pin "IPI" input
+			(at 162.56 91.44 0)
+			(effects
+				(font
+					(size 1.27 1.27)
+				)
+				(justify right)
+			)
+		)
+		(pin "DPO" output
+			(at 162.56 81.28 0)
+			(effects
+				(font
+					(size 1.27 1.27)
+				)
+				(justify right)
+			)
+		)

Commit message: Latest changes
Other:
- added sheet RSA_STAGE_MODULE1 (STAGE.kicad_sch)
- added sheet RSA_STAGE_MODULE2 (STAGE.kicad_sch)
- note added: "..."
